File: Production/SparkFun_LTE_Stick_LARA_R6-Panel.brd (EAGLE design)
At the start: 90.9 x 121.9 mm, 390 parts, among them IC1 SN74AVC4T774PW, IC2 SN74AVC4T774PW, IC3 SN74AVC4T774PW, IC4 SN74AVC4T774PW, IC5 SN74AVC4T774PW, IC6 SN74AVC4T774PW, J1 NANO_SIM, J10 NANO_SIM, J6 NANO_SIM, U1 LARA-R6401, U2 AP7361C-33, U3 LARA-R6401, U4 AP7361C-33, U5 LARA-R6401, U6 AP7361C-33

Commit message: Add v10 Panel
Parts:
- added C100, C48, C61, C74, C87: 100uF, SparkFun-Capacitors:PANASONIC_D
- added C101, C47, C49, C60, C62, C73, C75, C86, C88, C99: 10uF, SparkFun-Capacitors:0805
- added C102, C44, C45, C46, C50, C57, C58, C59, C63, C70, C71, C72, C76, C83, C84, C85, C89, C96, C97, C98: 0.1uF, SparkFun-Capacitors:0603
- added C103, C51, C64, C77, C90: 15pF, SparkFun-Capacitors:0603
- added C104, C52, C65, C78, C91: 68pF, SparkFun-Capacitors:0603
- added C40, C41, C42, C43, C53, C54, C55, C56, C66, C67, C68, C69, C79, C80, C81, C82, C92, C93, C94, C95: 47pF, SparkFun-Capacitors:0603
- added D31, D41, D51, D61, D71: PRTR5V0U2F, SparkFun-IC-Power:SOT886
- added D32, D33, D42, D43, D52, D53, D62, D63, D72, D73: PESD0402-0402, SparkFun-DiscreteSemi:0402
- added D34, D44, D54, D64, D74: DT1042-04SO-7, SparkFun-DiscreteSemi:SOT23-6L
- added D35, D36, D45, D46, D55, D56, D65, D66, D75, D76: Red, SparkFun-LED:LED-0603
- added D37, D38, D47, D48, D57, D58, D67, D68, D77, D78: 3A/10V/280mV, SparkFun-DiscreteSemi:SOD-323
- added D39, D40, D49, D50, D59, D60, D69, D70, D79, D80: 120mA/40V/370mV, SparkFun-DiscreteSemi:SOD-523
- added DTR3, DTR4, DTR5, DTR6, DTR7, ON_LED3, ON_LED4, ON_LED5, ON_LED6, ON_LED7, PWR_LED3, PWR_LED4, PWR_LED5, PWR_LED6, PWR_LED7, SHLD3, SHLD4, SHLD5, SHLD6, SHLD7: JUMPER-SMT_2_NC_TRACE_SILK, SparkFun-Jumpers:SMT-JUMPER_2_NC_TRACE_SILK
- added E10, E11, E12, E13, E14, E15, E16, E7, E8, E9: ANTENNA-SMA-GROUNDEDEDGE_SMA, SparkFun-RF:SMA-EDGE
- added F4, F5, F6, F7, F8: 6V/2A, SparkFun-Fuses:1210
- added FD13, FD14, FD15, FD16, FD17, FD18, FD19, FD20, FD21, FD22, FD23, FD24, FD25, FD26, FD27, FD28, FD29, FD30, FD31, FD32: FIDUCIAL1X2, SparkFun-Aesthetics:FIDUCIAL-1X2
- added H13, H14, H15, H16, H17, H18, H19, H20, H21, H22, H23, H24, H25, H26, H27, H28, H29, H30, H31, H32: STAND-OFF, SparkFun-Hardware:STAND-OFF
- added IC10, IC11, IC12, IC13, IC14, IC15, IC16, IC7, IC8, IC9: SN74AVC4T774PW, SparkFun-IC-Comms:SOP65P640X120-16N
- added J13, J17, J21, J25, J29: (no value), SparkFun-Connectors:USB-C-16P_4LAYER-PADS
- added J14, J18, J22, J26, J30: NANO_SIM, SparkFun-Connectors:NANO_SIM_PP
- added J15, J19, J23, J27, J31: (no value), SparkFun-Connectors:1X12_NO_SILK
- added J16, J20, J24, J28, J32: (no value), SparkFun-Connectors:1X04_NO_SILK
- added LOGO10, LOGO12, LOGO14, LOGO16, LOGO8: OSHW-LOGOM, SparkFun-Aesthetics:OSHW-LOGO-M
- added LOGO11, LOGO13, LOGO15, LOGO7, LOGO9: SFE_LOGO_NAME_FLAME.1_INCH, SparkFun-Aesthetics:SFE_LOGO_NAME_FLAME_.1
- added ON_BTN3, ON_BTN4, ON_BTN5, ON_BTN6, ON_BTN7, RST_BTN3, RST_BTN4, RST_BTN5, RST_BTN6, RST_BTN7: MOMENTARY-SWITCH-SPST-SMD-4.6X2.8MM, SparkFun-Switches:TACTILE_SWITCH_SMD_4.6X2.8MM
- added R22, R23, R29, R30, R36, R37, R43, R44, R50, R51: 5.1k, SparkFun-Resistors:0603
- added R24, R25, R28, R31, R32, R35, R38, R39, R42, R45, R46, R49, R52, R53, R56: 100k, SparkFun-Resistors:0603
- added R26, R33, R40, R47, R54: 4.7k, SparkFun-Resistors:0603
- added R27, R34, R41, R48, R55: 220, SparkFun-Resistors:0603
- added TP100, TP101, TP102, TP103, TP104, TP105, TP106, TP107, TP108, TP109, TP110, TP111, TP112, TP113, TP114, TP115, TP116, TP117, TP118, TP119, TP120, TP121, TP122, TP123, TP124, TP125, TP126, TP127, TP128, TP129, TP130, TP131, TP132, TP133, TP134, TP135, TP136, TP52, TP53, TP54, TP55, TP56, TP57, TP58, TP59, TP60, TP61, TP62, TP63, TP64, TP65, TP66, TP67, TP68, TP69, TP70, TP71, TP72, TP73, TP74, TP75, TP76, TP77, TP78, TP79, TP80, TP81, TP82, TP83, TP84, TP85, TP86, TP87, TP88, TP89, TP90, TP91, TP92, TP93, TP94, TP95, TP96, TP97, TP98, TP99: TEST-POINT3X5, SparkFun-Connectors:PAD.03X.05
- added U$163, U$220, U$277, U$334, U$391, U$448: (no value), output:3#3V0
- added U$164, U$221, U$278, U$335, U$392, U$449: (no value), output:UART20
- added U$165, U$222, U$279, U$336, U$393, U$450: (no value), output:GPIO0
- added U$166, U$223, U$280, U$337, U$394, U$451: (no value), output:I2C0
- added U$167, U$224, U$281, U$338, U$395, U$452: (no value), output:#_#ON##0
- added U$168, U$169, U$225, U$226, U$282, U$283, U$339, U$340, U$396, U$397, U$453, U$454: (no value), output:ON0
- added U$170, U$227, U$284, U$341, U$398, U$455: (no value), output:#ON_LED#0
- added U$171, U$228, U$285, U$342, U$399, U$456: (no value), output:#PWR_LED#0
- added U$172, U$189, U$229, U$246, U$286, U$303, U$343, U$360, U$400, U$417: (no value), output:LTE_STICK0
- added U$173, U$183, U$230, U$240, U$287, U$297, U$344, U$354, U$401, U$411: (no value), output:#_3V3#0
- added U$174, U$175, U$231, U$232, U$288, U$289, U$345, U$346, U$402, U$403: (no value), output:#_GND#0
- added U$176, U$177, U$233, U$234, U$290, U$291, U$347, U$348, U$404, U$405: (no value), output:#GND_#0
- added U$178, U$180, U$235, U$237, U$292, U$294, U$349, U$351, U$406, U$408: (no value), output:#3V3_#0
- added U$179, U$236, U$293, U$350, U$407: (no value), output:#VIN_#0
- added U$181, U$238, U$295, U$352, U$409: (no value), output:#1V8_#0
- added U$182, U$239, U$296, U$353, U$410: (no value), output:#_1V8#0
- added U$184, U$241, U$298, U$355, U$412: (no value), output:#_VIN#0
- added U$185, U$242, U$299, U$356, U$413: (no value), output:#_CTS#0
- added U$186, U$243, U$300, U$357, U$414: (no value), output:#_RTS#0
- added U$187, U$244, U$301, U$358, U$415: (no value), output:#_CLK#0
- added U$188, U$245, U$302, U$359, U$416: (no value), output:#_WA#0
- added U$190, U$247, U$304, U$361, U$418: (no value), output:#SHLD#0
- added U$191, U$248, U$305, U$362, U$419: (no value), output:#DTR#0
- added U$192, U$249, U$306, U$363, U$420: (no value), output:PWR0
- added U$193, U$250, U$307, U$364, U$421: (no value), output:#_#RST##0
- added U$194, U$251, U$308, U$365, U$422: (no value), SparkFun-Aesthetics:SFE_LOGO_FLAME_.2
- added U$195, U$196, U$252, U$253, U$309, U$310, U$366, U$367, U$423, U$424: (no value), output:LARA#R60
- added U$197, U$254, U$311, U$368, U$425: (no value), output:#RTS_#0
- added U$198, U$255, U$312, U$369, U$426: (no value), output:#CTS_#0
- added U$199, U$256, U$313, U$370, U$427: (no value), output:##RESET#_#0
- added U$200, U$257, U$314, U$371, U$428: (no value), output:##PWR_ON#_#0
- added U$201, U$258, U$315, U$372, U$429: (no value), output:#_RXA#0
- added U$202, U$259, U$316, U$373, U$430: (no value), output:#_TXA#0
- added U$203, U$260, U$317, U$374, U$431: (no value), output:#_TXD#0
- added U$204, U$261, U$318, U$375, U$432: (no value), output:#_RXD#0
- added U$205, U$262, U$319, U$376, U$433: (no value), output:#RXD_#0
- added U$206, U$263, U$320, U$377, U$434: (no value), output:#TXD_#0
- added U$207, U$264, U$321, U$378, U$435: (no value), output:#RXA_#0
- added U$208, U$265, U$322, U$379, U$436: (no value), output:#TXA_#0
- added U$209, U$266, U$323, U$380, U$437: (no value), output:#CLK_#0
- added U$210, U$267, U$324, U$381, U$438: (no value), output:#WA_#0
- added U$211, U$268, U$325, U$382, U$439: (no value), output:UART0
- added U$212, U$269, U$326, U$383, U$440: (no value), output:I2S0
- added U$213, U$270, U$327, U$384, U$441: (no value), output:ORIENTATION0
- added U$214, U$271, U$328, U$385, U$442: (no value), output:RST0
- added U$215, U$272, U$329, U$386, U$443: (no value), output:SIM_CARD0
- added U$216, U$273, U$330, U$387, U$444: (no value), output:VOLTAGE_LEVEL0
- added U$217, U$274, U$331, U$388, U$445: (no value), output:TEST_POINTS0
- added U$218, U$275, U$332, U$389, U$446: (no value), output:PTH_PADS0
- added U$219, U$276, U$333, U$390, U$447: (no value), output:1#8V0
- added U10, U12, U14, U16, U8: AP7361C-33, SparkFun-IC-Power:UDFN-8
- added U11, U13, U15, U7, U9: LARA-R6401, SparkFun-RF:LARA-LGA
- D15, D16, D25, D26, D5, D6: value (none) -> Red
- U$100: device output:ORIENTATION0 -> output:RST0
- U$101: device output:RST0 -> output:SIM_CARD0
- U$102: device output:PON0 -> output:VOLTAGE_LEVEL0
- U$103: device output:SIM_CARD0 -> output:TEST_POINTS0
- U$104: device output:VOLTAGE_LEVEL0 -> output:PTH_PADS0
- U$105: device output:TEST_POINTS0 -> output:1#8V0
- U$106: device output:PTH_PADS0 -> output:3#3V0
- U$107: device output:1#8V0 -> output:UART20
- U$108: device output:3#3V0 -> output:GPIO0
- U$109: device output:LTE_STICK0 -> output:I2C0
- U$110: device output:#_3V3#0 -> output:#_#ON##0
- U$111, U$112: device output:#_GND#0 -> output:ON0
- U$113: device output:#GND_#0 -> output:#ON_LED#0
- U$114, U$60: device output:#GND_#0 -> output:#PWR_LED#0
- U$115: device output:#3V3_#0 -> output:LTE_STICK0
- U$116: device output:#VIN_#0 -> output:#_3V3#0
- U$117, U$61: device output:#3V3_#0 -> output:#_GND#0
- U$118: device output:#1V8_#0 -> output:#_GND#0
- U$119: device output:#_1V8#0 -> output:#GND_#0
- U$120: device output:#_3V3#0 -> output:#GND_#0
- U$121: device output:#_VIN#0 -> output:#3V3_#0
- U$122: device output:#_CTS#0 -> output:#VIN_#0
- U$123: device output:#_RTS#0 -> output:#3V3_#0
- U$124: device output:#_CLK#0 -> output:#1V8_#0
- U$125: device output:#_WA#0 -> output:#_1V8#0
- U$126: device output:LTE_STICK0 -> output:#_3V3#0
- U$127: device output:#SHLD#0 -> output:#_VIN#0
- U$128: device output:#DTR#0 -> output:#_CTS#0
- U$129: device output:PWR0 -> output:#_RTS#0
- U$130: device output:#_#RST##0 -> output:#_CLK#0
- U$131: device SparkFun-Aesthetics:SFE_LOGO_FLAME_.2 -> output:#_WA#0
- U$132: device output:LARA#R60 -> output:LTE_STICK0
- U$133: device output:LARA#R60 -> output:#SHLD#0
- U$134: device output:#PWR#0 -> output:#DTR#0
- U$135: device output:#RTS_#0 -> output:PWR0
- U$136: device output:#CTS_#0 -> output:#_#RST##0
- U$137: device output:##RESET#_#0 -> SparkFun-Aesthetics:SFE_LOGO_FLAME_.2
- U$138: device output:#PON#0 -> output:LARA#R60
- U$139: device output:PON0 -> output:LARA#R60
- U$140: device output:#_#PON##0 -> output:#RTS_#0
- U$141: device output:##PWR_ON#_#0 -> output:#CTS_#0
- U$142: device output:#_RXA#0 -> output:##RESET#_#0
- U$143: device output:#_TXA#0 -> output:##PWR_ON#_#0
- U$144: device output:#_TXD#0 -> output:#_RXA#0
- U$145: device output:#_RXD#0 -> output:#_TXA#0
- U$146: device output:#RXD_#0 -> output:#_TXD#0
- U$147: device output:#TXD_#0 -> output:#_RXD#0
- U$148: device output:#RXA_#0 -> output:#RXD_#0
- U$149: device output:#TXA_#0 -> output:#TXD_#0
- U$150: device output:#CLK_#0 -> output:#RXA_#0
- U$151: device output:#WA_#0 -> output:#TXA_#0
- U$152: device output:UART0 -> output:#CLK_#0
- U$153: device output:I2S0 -> output:#WA_#0
- U$154: device output:ORIENTATION0 -> output:UART0
- U$155: device output:RST0 -> output:I2S0
- U$156: device output:PON0 -> output:ORIENTATION0
- U$157: device output:SIM_CARD0 -> output:RST0
- U$158: device output:VOLTAGE_LEVEL0 -> output:SIM_CARD0
- U$159: device output:TEST_POINTS0 -> output:VOLTAGE_LEVEL0
- U$160: device output:PTH_PADS0 -> output:TEST_POINTS0
- U$161: device output:1#8V0 -> output:PTH_PADS0
- U$162: device output:3#3V0 -> output:1#8V0
- U$29: device output:#_#PON##0 -> output:LTE_STICK0
- U$36: device output:#PWR#0 -> output:#_3V3#0
- U$37: device output:PON0 -> output:ON0
- U$39: device output:#PON#0 -> output:ON0
- U$53: device output:PON0 -> output:#ON_LED#0
- U$55: device output:LTE_STICK0 -> output:#_GND#0
- U$56: device output:#_3V3#0 -> output:UART20
- U$57: device output:#_GND#0 -> output:GPIO0
- U$58: device output:#_GND#0 -> output:I2C0
- U$59: device output:#GND_#0 -> output:#_#ON##0
- U$62: device output:#VIN_#0 -> output:#GND_#0
- U$63: device output:#3V3_#0 -> output:#GND_#0
- U$64: device output:#1V8_#0 -> output:#3V3_#0
- U$65: device output:#_1V8#0 -> output:#VIN_#0
- U$66: device output:#_3V3#0 -> output:#3V3_#0
- U$67: device output:#_VIN#0 -> output:#1V8_#0
- U$68: device output:#_CTS#0 -> output:#_1V8#0
- U$69: device output:#_RTS#0 -> output:#_3V3#0
- U$70: device output:#_CLK#0 -> output:#_VIN#0
- U$71: device output:#_WA#0 -> output:#_CTS#0
- U$72: device output:LTE_STICK0 -> output:#_RTS#0
- U$73: device output:#SHLD#0 -> output:#_CLK#0
- U$74: device output:#DTR#0 -> output:#_WA#0
- U$75: device output:PWR0 -> output:LTE_STICK0
- U$76: device output:#_#RST##0 -> output:#SHLD#0
- U$77: device SparkFun-Aesthetics:SFE_LOGO_FLAME_.2 -> output:#DTR#0
- U$78: device output:LARA#R60 -> output:PWR0
- U$79: device output:LARA#R60 -> output:#_#RST##0
- U$80: device output:#PWR#0 -> SparkFun-Aesthetics:SFE_LOGO_FLAME_.2
- U$81: device output:#RTS_#0 -> output:LARA#R60
- U$82: device output:#CTS_#0 -> output:LARA#R60
- U$83: device output:##RESET#_#0 -> output:#RTS_#0
- U$84: device output:#PON#0 -> output:#CTS_#0
- U$85: device output:PON0 -> output:##RESET#_#0
- U$86: device output:#_#PON##0 -> output:##PWR_ON#_#0
- U$87: device output:##PWR_ON#_#0 -> output:#_RXA#0
- U$88: device output:#_RXA#0 -> output:#_TXA#0
- U$89: device output:#_TXA#0 -> output:#_TXD#0
- U$90: device output:#_TXD#0 -> output:#_RXD#0
- U$91: device output:#_RXD#0 -> output:#RXD_#0
- U$92: device output:#RXD_#0 -> output:#TXD_#0
- U$93: device output:#TXD_#0 -> output:#RXA_#0
- U$94: device output:#RXA_#0 -> output:#TXA_#0
- U$95: device output:#TXA_#0 -> output:#CLK_#0
- U$96: device output:#CLK_#0 -> output:#WA_#0
- U$97: device output:#WA_#0 -> output:UART0
- U$98: device output:UART0 -> output:I2S0
- U$99: device output:I2S0 -> output:ORIENTATION0
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- renumbered PON to ON_LED, PON1 to ON_LED1, PON2 to ON_LED2, PWR to PWR_LED, PWR1 to PWR_LED1, PWR2 to PWR_LED2, S1 to ON_BTN, S2 to RST_BTN, S3 to ON_BTN1, S4 to RST_BTN1, S5 to ON_BTN2, S6 to RST_BTN2
Connections:
- new net !PWR_ON!3: D39.A, ON_BTN3.3, ON_BTN3.4, U7.15
- new net !PWR_ON!4: D49.A, ON_BTN4.3, ON_BTN4.4, U9.15
- new net !PWR_ON!5: D59.A, ON_BTN5.3, ON_BTN5.4, U11.15
- new net !PWR_ON!6: D69.A, ON_BTN6.3, ON_BTN6.4, U13.15
- new net !PWR_ON!7: D79.A, ON_BTN7.3, ON_BTN7.4, U15.15
- new net !RESET!3: D40.A, RST_BTN3.3, RST_BTN3.4, U7.18
- new net !RESET!4: D50.A, RST_BTN4.3, RST_BTN4.4, U9.18
- new net !RESET!5: D60.A, RST_BTN5.3, RST_BTN5.4, U11.18
- new net !RESET!6: D70.A, RST_BTN6.3, RST_BTN6.4, U13.18
- new net !RESET!7: D80.A, RST_BTN7.3, RST_BTN7.4, U15.18
- new net 1.8V3: C45.1, C46.1, IC7.1, IC7.16, IC7.7, IC8.1, IC8.16, IC8.2, IC8.7, J16.4, ON_LED3.2, R24.2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
- new net 1.8V4: C58.1, C59.1, IC10.1, IC10.16, IC10.2, IC10.7, IC9.1, IC9.16, IC9.7, J20.4, ON_LED4.2, R31.2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
- new net 1.8V5: C71.1, C72.1, IC11.1, IC11.16, IC11.7, IC12.1, IC12.16, IC12.2, IC12.7, J24.4, ON_LED5.2, R38.2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
- new net 1.8V6: C84.1, C85.1, IC13.1, IC13.16, IC13.7, IC14.1, IC14.16, IC14.2, IC14.7, J28.4, ON_LED6.2, R45.2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
- new net 1.8V7: C97.1, C98.1, IC15.1, IC15.16, IC15.7, IC16.1, IC16.16, IC16.2, IC16.7, J32.4, ON_LED7.2, R52.2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
- new net 3.3V3: C48.+, C49.1, C50.1, C51.1, C52.1, IC7.15, IC8.15, J15.6, J16.3, PWR_LED3.2, U7.51, U7.52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
- new net 3.3V4: C61.+, C62.1, C63.1, C64.1, C65.1, IC10.15, IC9.15, J19.6, J20.3, PWR_LED4.2, U10.1, U9.51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
- new net 3.3V5: C74.+, C75.1, C76.1, C77.1, C78.1, IC11.15, IC12.15, J23.6, J24.3, PWR_LED5.2, U11.51, U11.52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
- new net 3.3V6: C87.+, C88.1, C89.1, C90.1, C91.1, IC13.15, IC14.15, J27.6, J28.3, PWR_LED6.2, U13.51, U13.52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
- new net 3.3V7: C100.+, C101.1, C102.1, C103.1, C104.1, IC15.15, IC16.15, J31.6, J32.3, PWR_LED7.2, U15.51, U15.52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
- new net 5V3: D37.A, F4.2
- new net 5V4: D47.A, F5.2
- new net 5V5: D57.A, F6.2
- new net 5V6: D67.A, F7.2
- new net 5V7: D77.A, F8.2
- new net ANT10: D43.1, E9.SIG, U9.62
- new net ANT11: D52.1, E12.SIG, U11.56
- new net ANT12: D53.1, E11.SIG, U11.62
- new net ANT13: D62.1, E14.SIG, U13.56
- new net ANT14: D63.1, E13.SIG, U13.62
- new net ANT15: D72.1, E16.SIG, U15.56
- new net ANT16: D73.1, E15.SIG, U15.62
- new net ANT7: D32.1, E8.SIG, U7.56
- new net ANT8: D33.1, E7.SIG, U7.62
- new net ANT9: D42.1, E10.SIG, U9.56
- new net CTS_10: IC11.12, J23.9
- new net CTS_11: IC13.5, U13.11
- new net CTS_12: IC13.12, J27.9
- new net CTS_13: IC15.5, U15.11
- new net CTS_14: IC15.12, J31.9
- new net CTS_5: IC7.5, U7.11
- new net CTS_6: IC7.12, J15.9
- new net CTS_7: IC9.5, U9.11
- new net CTS_8: IC9.12, J19.9
- new net CTS_9: IC11.5, U11.11
- new net DCD/RXD2_3: TP58.1, U7.8
- new net DCD/RXD2_4: TP75.1, U9.8
- new net DCD/RXD2_5: TP92.1, U11.8
- new net DCD/RXD2_6: TP109.1, U13.8
- new net DCD/RXD2_7: TP126.1, U15.8
- new net DSR/RTS2_3: TP56.1, U7.6
- new net DSR/RTS2_4: TP73.1, U9.6
- new net DSR/RTS2_5: TP90.1, U11.6
- new net DSR/RTS2_6: TP107.1, U13.6
- new net DSR/RTS2_7: TP124.1, U15.6
- new net DTR/TXD2_3: DTR3.2, TP59.1, U7.9
- new net DTR/TXD2_4: DTR4.2, TP76.1, U9.9
- new net DTR/TXD2_5: DTR5.2, TP93.1, U11.9
- new net DTR/TXD2_6: DTR6.2, TP110.1, U13.9
- new net DTR/TXD2_7: DTR7.2, TP127.1, U15.9
- new net EN3: R25.1, U8.5
- new net EN4: R32.1, U10.5
- new net EN5: R39.1, U12.5
- new net EN6: R46.1, U14.5
- new net EN7: R53.1, U16.5
- new net GND3: C40.2, C41.2, C42.2, C43.2, C44.2, C45.2, C46.2, C47.2, C48.-, C49.2, C50.2, C51.2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
- new net GND4: C53.2, C54.2, C55.2, C56.2, C57.2, C58.2, C59.2, C60.2, C61.-, C62.2, C63.2, C64.2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
- new net GND5: C66.2, C67.2, C68.2, C69.2, C70.2, C71.2, C72.2, C73.2, C74.-, C75.2, C76.2, C77.2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
- new net GND6: C79.2, C80.2, C81.2, C82.2, C83.2, C84.2, C85.2, C86.2, C87.-, C88.2, C89.2, C90.2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
- new net GND7: C100.-, C101.2, C102.2, C103.2, C104.2, C92.2, C93.2, C94.2, C95.2, C96.2, C97.2, C98.2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
- new net I2S_CLK_10: IC12.5, U11.36
- new net I2S_CLK_11: IC14.12, J27.3
- new net I2S_CLK_12: IC14.5, U13.36
- new net I2S_CLK_13: IC16.12, J31.3
- new net I2S_CLK_14: IC16.5, U15.36
- new net I2S_CLK_5: IC8.12, J15.3
- new net I2S_CLK_6: IC8.5, U7.36
- new net I2S_CLK_7: IC10.12, J19.3
- new net I2S_CLK_8: IC10.5, U9.36
- new net I2S_CLK_9: IC12.12, J23.3
- new net I2S_RXA_10: IC12.6, U11.37
- new net I2S_RXA_11: IC14.11, J27.4
- new net I2S_RXA_12: IC14.6, U13.37
- new net I2S_RXA_13: IC16.11, J31.4
- new net I2S_RXA_14: IC16.6, U15.37
- new net I2S_RXA_5: IC8.11, J15.4
- new net I2S_RXA_6: IC8.6, U7.37
- new net I2S_RXA_7: IC10.11, J19.4
- new net I2S_RXA_8: IC10.6, U9.37
- new net I2S_RXA_9: IC12.11, J23.4
- new net I2S_TXA_10: IC12.4, U11.35
- new net I2S_TXA_11: IC14.13, J27.2
- new net I2S_TXA_12: IC14.4, U13.35
- new net I2S_TXA_13: IC16.13, J31.2
- new net I2S_TXA_14: IC16.4, U15.35
- new net I2S_TXA_5: IC8.13, J15.2
- new net I2S_TXA_6: IC8.4, U7.35
- new net I2S_TXA_7: IC10.13, J19.2
- new net I2S_TXA_8: IC10.4, U9.35
- new net I2S_TXA_9: IC12.13, J23.2
- new net I2S_WA_10: IC12.3, U11.34
- new net I2S_WA_11: IC14.14, J27.1
- new net I2S_WA_12: IC14.3, U13.34
- new net I2S_WA_13: IC16.14, J31.1
- new net I2S_WA_14: IC16.3, U15.34
- new net I2S_WA_5: IC8.14, J15.1
- new net I2S_WA_6: IC8.3, U7.34
- new net I2S_WA_7: IC10.14, J19.1
- new net I2S_WA_8: IC10.3, U9.34
- new net I2S_WA_9: IC12.14, J23.1
- new net IO1_3: TP62.1, U7.16
- new net IO1_4: TP79.1, U9.16
- new net IO1_5: TP96.1, U11.16
- new net IO1_6: TP113.1, U13.16
- new net IO1_7: TP130.1, U15.16
- new net IO2_3: TP63.1, U7.23
- new net IO2_4: TP80.1, U9.23
- new net IO2_5: TP97.1, U11.23
- new net IO2_6: TP114.1, U13.23
- new net IO2_7: TP131.1, U15.23
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Routing:
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- added copper zone on layer 15, net 1.8V3
- added copper zone on layer 15, net 1.8V4
- added copper zone on layer 15, net 1.8V5
- added copper zone on layer 15, net 1.8V6
- added copper zone on layer 15, net 1.8V7
- added copper zone on layer 1, net 3.3V3
- added copper zone on layer 15, net 3.3V3
- added copper zone on layer 1, net 3.3V4
- added copper zone on layer 15, net 3.3V4
- added copper zone on layer 1, net 3.3V5
- added copper zone on layer 15, net 3.3V5
- added copper zone on layer 1, net 3.3V6
- added copper zone on layer 15, net 3.3V6
- added copper zone on layer 1, net 3.3V7
- added copper zone on layer 15, net 3.3V7
- added copper zone on layer 1, net GND3
- added copper zone on layer 16, net GND3
- added copper zone on layer 2, net GND3
- added copper zone on layer 1, net GND4
- added copper zone on layer 16, net GND4
- added copper zone on layer 2, net GND4
- added copper zone on layer 1, net GND5
- added copper zone on layer 16, net GND5
- added copper zone on layer 2, net GND5
- added copper zone on layer 1, net GND6
- added copper zone on layer 16, net GND6
- added copper zone on layer 2, net GND6
- added copper zone on layer 1, net GND7
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Other:
- board size 90.9 x 121.9 mm -> 116.8 x 188 mm
- board text added: "v10"
- board text removed: "v01"

Commit message: v11 - Label SMA connectors in silkscreen
Parts:
- added U$457: (no value), output:#_RXA#0
- added U$458: (no value), output:#_TXA#0
- added U$459: (no value), output:#_TXD#0
- added U$460: (no value), output:#_RXD#0
- added U$461: (no value), output:#RXD_#0
- added U$462: (no value), output:#TXD_#0
- added U$463: (no value), output:#RXA_#0
- added U$464: (no value), output:#TXA_#0
- added U$465: (no value), output:#CLK_#0
- added U$466: (no value), output:#WA_#0
- added U$467: (no value), output:UART0
- added U$468: (no value), output:I2S0
- added U$469: (no value), output:ORIENTATION0
- added U$470: (no value), output:RST0
- added U$471: (no value), output:SIM_CARD0
- added U$472: (no value), output:VOLTAGE_LEVEL0
- added U$473: (no value), output:TEST_POINTS0
- added U$474: (no value), output:PTH_PADS0
- added U$475: (no value), output:1#8V0
- added U$476: (no value), output:3#3V0
- added U$477: (no value), output:UART20
- added U$478: (no value), output:GPIO0
- added U$479: (no value), output:I2C0
- added U$480: (no value), output:#_#ON##0
- added U$481, U$482: (no value), output:ON0
- added U$483: (no value), output:#ON_LED#0
- added U$484: (no value), output:#PWR_LED#0
- added U$485, U$486: (no value), output:ANT10
- added U$487, U$488: (no value), output:ANT20
- U$100: device output:RST0 -> output:#WA_#0
- U$101: device output:SIM_CARD0 -> output:UART0
- U$102: device output:VOLTAGE_LEVEL0 -> output:I2S0
- U$103: device output:TEST_POINTS0 -> output:ORIENTATION0
- U$104: device output:PTH_PADS0 -> output:RST0
- U$105: device output:1#8V0 -> output:SIM_CARD0
- U$106: device output:3#3V0 -> output:VOLTAGE_LEVEL0
- U$107: device output:UART20 -> output:TEST_POINTS0
- U$108: device output:GPIO0 -> output:PTH_PADS0
- U$109: device output:I2C0 -> output:1#8V0
- U$110: device output:#_#ON##0 -> output:3#3V0
- U$111: device output:ON0 -> output:UART20
- U$112: device output:ON0 -> output:GPIO0
- U$113: device output:#ON_LED#0 -> output:I2C0
- U$114: device output:#PWR_LED#0 -> output:#_#ON##0
- U$115, U$360: device output:LTE_STICK0 -> output:ON0
- U$116: device output:#_3V3#0 -> output:ON0
- U$117: device output:#_GND#0 -> output:#ON_LED#0
- U$118: device output:#_GND#0 -> output:#PWR_LED#0
- U$119, U$120: device output:#GND_#0 -> output:ANT10
- U$121: device output:#3V3_#0 -> output:ANT20
- U$122: device output:#VIN_#0 -> output:ANT20
- U$123: device output:#3V3_#0 -> output:LTE_STICK0
- U$124: device output:#1V8_#0 -> output:#_3V3#0
- U$125: device output:#_1V8#0 -> output:#_GND#0
- U$126: device output:#_3V3#0 -> output:#_GND#0
- U$127: device output:#_VIN#0 -> output:#GND_#0
- U$128: device output:#_CTS#0 -> output:#GND_#0
- U$129: device output:#_RTS#0 -> output:#3V3_#0
- U$130: device output:#_CLK#0 -> output:#VIN_#0
- U$131: device output:#_WA#0 -> output:#3V3_#0
- U$132: device output:LTE_STICK0 -> output:#1V8_#0
- U$133: device output:#SHLD#0 -> output:#_1V8#0
- U$134: device output:#DTR#0 -> output:#_3V3#0
- U$135: device output:PWR0 -> output:#_VIN#0
- U$136: device output:#_#RST##0 -> output:#_CTS#0
- U$137: device SparkFun-Aesthetics:SFE_LOGO_FLAME_.2 -> output:#_RTS#0
- U$138: device output:LARA#R60 -> output:#_CLK#0
- U$139: device output:LARA#R60 -> output:#_WA#0
- U$140: device output:#RTS_#0 -> output:LTE_STICK0
- U$141: device output:#CTS_#0 -> output:#SHLD#0
- U$142: device output:##RESET#_#0 -> output:#DTR#0
- U$143: device output:##PWR_ON#_#0 -> output:PWR0
- U$144: device output:#_RXA#0 -> output:#_#RST##0
- U$145: device output:#_TXA#0 -> SparkFun-Aesthetics:SFE_LOGO_FLAME_.2
- U$146: device output:#_TXD#0 -> output:LARA#R60
- U$147: device output:#_RXD#0 -> output:LARA#R60
- U$148: device output:#RXD_#0 -> output:#RTS_#0
- U$149: device output:#TXD_#0 -> output:#CTS_#0
- U$150: device output:#RXA_#0 -> output:##RESET#_#0
- U$151: device output:#TXA_#0 -> output:##PWR_ON#_#0
- U$152: device output:#CLK_#0 -> output:#_RXA#0
- U$153: device output:#WA_#0 -> output:#_TXA#0
- U$154: device output:UART0 -> output:#_TXD#0
- U$155: device output:I2S0 -> output:#_RXD#0
- U$156: device output:ORIENTATION0 -> output:#RXD_#0
- U$157: device output:RST0 -> output:#TXD_#0
- U$158: device output:SIM_CARD0 -> output:#RXA_#0
- U$159: device output:VOLTAGE_LEVEL0 -> output:#TXA_#0
- U$160: device output:TEST_POINTS0 -> output:#CLK_#0
- U$161: device output:PTH_PADS0 -> output:#WA_#0
- U$162: device output:1#8V0 -> output:UART0
- U$163: device output:3#3V0 -> output:I2S0
- U$164: device output:UART20 -> output:ORIENTATION0
- U$165: device output:GPIO0 -> output:RST0
- U$166: device output:I2C0 -> output:SIM_CARD0
- U$167: device output:#_#ON##0 -> output:VOLTAGE_LEVEL0
- U$168: device output:ON0 -> output:TEST_POINTS0
- U$169: device output:ON0 -> output:PTH_PADS0
- U$170: device output:#ON_LED#0 -> output:1#8V0
- U$171: device output:#PWR_LED#0 -> output:3#3V0
- U$172: device output:LTE_STICK0 -> output:UART20
- U$173: device output:#_3V3#0 -> output:GPIO0
- U$174: device output:#_GND#0 -> output:I2C0
- U$175: device output:#_GND#0 -> output:#_#ON##0
- U$176, U$177: device output:#GND_#0 -> output:ON0
- U$178: device output:#3V3_#0 -> output:#ON_LED#0
- U$179: device output:#VIN_#0 -> output:#PWR_LED#0
- U$180: device output:#3V3_#0 -> output:ANT10
- U$181: device output:#1V8_#0 -> output:ANT10
- U$182: device output:#_1V8#0 -> output:ANT20
- U$183: device output:#_3V3#0 -> output:ANT20
- U$184: device output:#_VIN#0 -> output:LTE_STICK0
- U$185: device output:#_CTS#0 -> output:#_3V3#0
- U$186: device output:#_RTS#0 -> output:#_GND#0
- U$187: device output:#_CLK#0 -> output:#_GND#0
- U$188: device output:#_WA#0 -> output:#GND_#0
- U$189: device output:LTE_STICK0 -> output:#GND_#0
- U$190: device output:#SHLD#0 -> output:#3V3_#0
- U$191: device output:#DTR#0 -> output:#VIN_#0
- U$192: device output:PWR0 -> output:#3V3_#0
- U$193: device output:#_#RST##0 -> output:#1V8_#0
- U$194: device SparkFun-Aesthetics:SFE_LOGO_FLAME_.2 -> output:#_1V8#0
- U$195: device output:LARA#R60 -> output:#_3V3#0
- U$196: device output:LARA#R60 -> output:#_VIN#0
- U$197: device output:#RTS_#0 -> output:#_CTS#0
- U$198: device output:#CTS_#0 -> output:#_RTS#0
- U$199: device output:##RESET#_#0 -> output:#_CLK#0
- U$200: device output:##PWR_ON#_#0 -> output:#_WA#0
- U$201: device output:#_RXA#0 -> output:LTE_STICK0
- U$202: device output:#_TXA#0 -> output:#SHLD#0
- U$203: device output:#_TXD#0 -> output:#DTR#0
- U$204: device output:#_RXD#0 -> output:PWR0
- U$205: device output:#RXD_#0 -> output:#_#RST##0
- U$206: device output:#TXD_#0 -> SparkFun-Aesthetics:SFE_LOGO_FLAME_.2
- U$207: device output:#RXA_#0 -> output:LARA#R60
- U$208: device output:#TXA_#0 -> output:LARA#R60
- U$209: device output:#CLK_#0 -> output:#RTS_#0
- U$210: device output:#WA_#0 -> output:#CTS_#0
- U$211: device output:UART0 -> output:##RESET#_#0
- U$212: device output:I2S0 -> output:##PWR_ON#_#0
- U$213: device output:ORIENTATION0 -> output:#_RXA#0
- U$214: device output:RST0 -> output:#_TXA#0
- U$215: device output:SIM_CARD0 -> output:#_TXD#0
- U$216: device output:VOLTAGE_LEVEL0 -> output:#_RXD#0
- U$217: device output:TEST_POINTS0 -> output:#RXD_#0
- U$218: device output:PTH_PADS0 -> output:#TXD_#0
- U$219: device output:1#8V0 -> output:#RXA_#0
- U$220: device output:3#3V0 -> output:#TXA_#0
- U$221: device output:UART20 -> output:#CLK_#0
- U$222: device output:GPIO0 -> output:#WA_#0
- U$223: device output:I2C0 -> output:UART0
- U$224: device output:#_#ON##0 -> output:I2S0
- U$225: device output:ON0 -> output:ORIENTATION0
- U$226: device output:ON0 -> output:RST0
- U$227: device output:#ON_LED#0 -> output:SIM_CARD0
- U$228: device output:#PWR_LED#0 -> output:VOLTAGE_LEVEL0
- U$229: device output:LTE_STICK0 -> output:TEST_POINTS0
- U$230: device output:#_3V3#0 -> output:PTH_PADS0
- U$231: device output:#_GND#0 -> output:1#8V0
- U$232: device output:#_GND#0 -> output:3#3V0
- U$233: device output:#GND_#0 -> output:UART20
- U$234: device output:#GND_#0 -> output:GPIO0
- U$235: device output:#3V3_#0 -> output:I2C0
- U$236: device output:#VIN_#0 -> output:#_#ON##0
- U$237: device output:#3V3_#0 -> output:ON0
- U$238: device output:#1V8_#0 -> output:ON0
- U$239: device output:#_1V8#0 -> output:#ON_LED#0
- U$240: device output:#_3V3#0 -> output:#PWR_LED#0
- U$241: device output:#_VIN#0 -> output:ANT10
- U$242: device output:#_CTS#0 -> output:ANT10
- U$243: device output:#_RTS#0 -> output:ANT20
- U$244: device output:#_CLK#0 -> output:ANT20
- U$245: device output:#_WA#0 -> output:LTE_STICK0
- U$246: device output:LTE_STICK0 -> output:#_3V3#0
- U$247: device output:#SHLD#0 -> output:#_GND#0
- U$248: device output:#DTR#0 -> output:#_GND#0
- U$249: device output:PWR0 -> output:#GND_#0
- U$250: device output:#_#RST##0 -> output:#GND_#0
- U$251: device SparkFun-Aesthetics:SFE_LOGO_FLAME_.2 -> output:#3V3_#0
- U$252: device output:LARA#R60 -> output:#VIN_#0
- U$253: device output:LARA#R60 -> output:#3V3_#0
- U$254: device output:#RTS_#0 -> output:#1V8_#0
- U$255: device output:#CTS_#0 -> output:#_1V8#0
- U$256: device output:##RESET#_#0 -> output:#_3V3#0
- U$257: device output:##PWR_ON#_#0 -> output:#_VIN#0
- U$258: device output:#_RXA#0 -> output:#_CTS#0
- U$259: device output:#_TXA#0 -> output:#_RTS#0
- U$260: device output:#_TXD#0 -> output:#_CLK#0
- U$261: device output:#_RXD#0 -> output:#_WA#0
- U$262: device output:#RXD_#0 -> output:LTE_STICK0
- U$263: device output:#TXD_#0 -> output:#SHLD#0
- U$264: device output:#RXA_#0 -> output:#DTR#0
- U$265: device output:#TXA_#0 -> output:PWR0
- U$266: device output:#CLK_#0 -> output:#_#RST##0
- U$267: device output:#WA_#0 -> SparkFun-Aesthetics:SFE_LOGO_FLAME_.2
- U$268: device output:UART0 -> output:LARA#R60
- U$269: device output:I2S0 -> output:LARA#R60
- U$270: device output:ORIENTATION0 -> output:#RTS_#0
- U$271: device output:RST0 -> output:#CTS_#0
- U$272: device output:SIM_CARD0 -> output:##RESET#_#0
- U$273: device output:VOLTAGE_LEVEL0 -> output:##PWR_ON#_#0
- U$274: device output:TEST_POINTS0 -> output:#_RXA#0
- U$275: device output:PTH_PADS0 -> output:#_TXA#0
- U$276: device output:1#8V0 -> output:#_TXD#0
- U$277: device output:3#3V0 -> output:#_RXD#0
- U$278: device output:UART20 -> output:#RXD_#0
- U$279: device output:GPIO0 -> output:#TXD_#0
- U$280: device output:I2C0 -> output:#RXA_#0
- U$281: device output:#_#ON##0 -> output:#TXA_#0
- U$282: device output:ON0 -> output:#CLK_#0
- U$283: device output:ON0 -> output:#WA_#0
- U$284: device output:#ON_LED#0 -> output:UART0
- U$285: device output:#PWR_LED#0 -> output:I2S0
- U$286: device output:LTE_STICK0 -> output:ORIENTATION0
- U$287: device output:#_3V3#0 -> output:RST0
- U$288: device output:#_GND#0 -> output:SIM_CARD0
- U$289: device output:#_GND#0 -> output:VOLTAGE_LEVEL0
- U$29, U$303: device output:LTE_STICK0 -> output:ANT10
- U$290: device output:#GND_#0 -> output:TEST_POINTS0
- U$291: device output:#GND_#0 -> output:PTH_PADS0
- U$292: device output:#3V3_#0 -> output:1#8V0
- U$293: device output:#VIN_#0 -> output:3#3V0
- U$294: device output:#3V3_#0 -> output:UART20
- U$295: device output:#1V8_#0 -> output:GPIO0
- U$296: device output:#_1V8#0 -> output:I2C0
- U$297: device output:#_3V3#0 -> output:#_#ON##0
- U$298: device output:#_VIN#0 -> output:ON0
- U$299: device output:#_CTS#0 -> output:ON0
- U$300: device output:#_RTS#0 -> output:#ON_LED#0
- U$301: device output:#_CLK#0 -> output:#PWR_LED#0
- U$302: device output:#_WA#0 -> output:ANT10
- U$304: device output:#SHLD#0 -> output:ANT20
- U$305: device output:#DTR#0 -> output:ANT20
- U$306: device output:PWR0 -> output:LTE_STICK0
- U$307: device output:#_#RST##0 -> output:#_3V3#0
- U$308: device SparkFun-Aesthetics:SFE_LOGO_FLAME_.2 -> output:#_GND#0
- U$309: device output:LARA#R60 -> output:#_GND#0
- U$310: device output:LARA#R60 -> output:#GND_#0
- U$311: device output:#RTS_#0 -> output:#GND_#0
- U$312: device output:#CTS_#0 -> output:#3V3_#0
- U$313: device output:##RESET#_#0 -> output:#VIN_#0
- U$314: device output:##PWR_ON#_#0 -> output:#3V3_#0
- U$315: device output:#_RXA#0 -> output:#1V8_#0
- U$316: device output:#_TXA#0 -> output:#_1V8#0
- U$317: device output:#_TXD#0 -> output:#_3V3#0
- U$318: device output:#_RXD#0 -> output:#_VIN#0
- U$319: device output:#RXD_#0 -> output:#_CTS#0
- U$320: device output:#TXD_#0 -> output:#_RTS#0
- U$321: device output:#RXA_#0 -> output:#_CLK#0
- U$322: device output:#TXA_#0 -> output:#_WA#0
- U$323: device output:#CLK_#0 -> output:LTE_STICK0
- U$324: device output:#WA_#0 -> output:#SHLD#0
- U$325: device output:UART0 -> output:#DTR#0
- U$326: device output:I2S0 -> output:PWR0
- U$327: device output:ORIENTATION0 -> output:#_#RST##0
- U$328: device output:RST0 -> SparkFun-Aesthetics:SFE_LOGO_FLAME_.2
- U$329: device output:SIM_CARD0 -> output:LARA#R60
- U$330: device output:VOLTAGE_LEVEL0 -> output:LARA#R60
- U$331: device output:TEST_POINTS0 -> output:#RTS_#0
- U$332: device output:PTH_PADS0 -> output:#CTS_#0
- U$333: device output:1#8V0 -> output:##RESET#_#0
- U$334: device output:3#3V0 -> output:##PWR_ON#_#0
- U$335: device output:UART20 -> output:#_RXA#0
- U$336: device output:GPIO0 -> output:#_TXA#0
- U$337: device output:I2C0 -> output:#_TXD#0
- U$338: device output:#_#ON##0 -> output:#_RXD#0
- U$339: device output:ON0 -> output:#RXD_#0
- U$340: device output:ON0 -> output:#TXD_#0
- U$341: device output:#ON_LED#0 -> output:#RXA_#0
- U$342: device output:#PWR_LED#0 -> output:#TXA_#0
- U$343: device output:LTE_STICK0 -> output:#CLK_#0
- U$344: device output:#_3V3#0 -> output:#WA_#0
- U$345: device output:#_GND#0 -> output:UART0
- U$346: device output:#_GND#0 -> output:I2S0
- U$347: device output:#GND_#0 -> output:ORIENTATION0
- U$348: device output:#GND_#0 -> output:RST0
- U$349: device output:#3V3_#0 -> output:SIM_CARD0
- U$350: device output:#VIN_#0 -> output:VOLTAGE_LEVEL0
- U$351: device output:#3V3_#0 -> output:TEST_POINTS0
- U$352: device output:#1V8_#0 -> output:PTH_PADS0
- U$353: device output:#_1V8#0 -> output:1#8V0
- U$354: device output:#_3V3#0 -> output:3#3V0
- U$355: device output:#_VIN#0 -> output:UART20
- U$356: device output:#_CTS#0 -> output:GPIO0
- U$357: device output:#_RTS#0 -> output:I2C0
- U$358: device output:#_CLK#0 -> output:#_#ON##0
- U$359: device output:#_WA#0 -> output:ON0
- U$36: device output:#_3V3#0 -> output:ANT10
- U$361: device output:#SHLD#0 -> output:#ON_LED#0
- U$362: device output:#DTR#0 -> output:#PWR_LED#0
- U$363: device output:PWR0 -> output:ANT10
- U$364: device output:#_#RST##0 -> output:ANT10
- U$365: device SparkFun-Aesthetics:SFE_LOGO_FLAME_.2 -> output:ANT20
- U$366: device output:LARA#R60 -> output:ANT20
- U$367: device output:LARA#R60 -> output:LTE_STICK0
- U$368: device output:#RTS_#0 -> output:#_3V3#0
- U$369: device output:#CTS_#0 -> output:#_GND#0
- U$370: device output:##RESET#_#0 -> output:#_GND#0
- U$371: device output:##PWR_ON#_#0 -> output:#GND_#0
- U$372: device output:#_RXA#0 -> output:#GND_#0
- U$373: device output:#_TXA#0 -> output:#3V3_#0
- U$374: device output:#_TXD#0 -> output:#VIN_#0
- U$375: device output:#_RXD#0 -> output:#3V3_#0
- U$376: device output:#RXD_#0 -> output:#1V8_#0
- U$377: device output:#TXD_#0 -> output:#_1V8#0
- U$378: device output:#RXA_#0 -> output:#_3V3#0
- U$379: device output:#TXA_#0 -> output:#_VIN#0
- U$380: device output:#CLK_#0 -> output:#_CTS#0
- U$381: device output:#WA_#0 -> output:#_RTS#0
- U$382: device output:UART0 -> output:#_CLK#0
- U$383: device output:I2S0 -> output:#_WA#0
- U$384: device output:ORIENTATION0 -> output:LTE_STICK0
- U$385: device output:RST0 -> output:#SHLD#0
- U$386: device output:SIM_CARD0 -> output:#DTR#0
- U$387: device output:VOLTAGE_LEVEL0 -> output:PWR0
- U$388: device output:TEST_POINTS0 -> output:#_#RST##0
- U$389: device output:PTH_PADS0 -> SparkFun-Aesthetics:SFE_LOGO_FLAME_.2
- U$390: device output:1#8V0 -> output:LARA#R60
- U$391: device output:3#3V0 -> output:LARA#R60
- U$392: device output:UART20 -> output:#RTS_#0
- U$393: device output:GPIO0 -> output:#CTS_#0
- U$394: device output:I2C0 -> output:##RESET#_#0
- U$395: device output:#_#ON##0 -> output:##PWR_ON#_#0
- U$396: device output:ON0 -> output:#_RXA#0
- U$397: device output:ON0 -> output:#_TXA#0
- U$398: device output:#ON_LED#0 -> output:#_TXD#0
- U$399: device output:#PWR_LED#0 -> output:#_RXD#0
- U$400: device output:LTE_STICK0 -> output:#RXD_#0
- U$401: device output:#_3V3#0 -> output:#TXD_#0
- U$402: device output:#_GND#0 -> output:#RXA_#0
- U$403: device output:#_GND#0 -> output:#TXA_#0
- U$404: device output:#GND_#0 -> output:#CLK_#0
- U$405: device output:#GND_#0 -> output:#WA_#0
- U$406: device output:#3V3_#0 -> output:UART0
- U$407: device output:#VIN_#0 -> output:I2S0
- U$408: device output:#3V3_#0 -> output:ORIENTATION0
- U$409: device output:#1V8_#0 -> output:RST0
- U$410: device output:#_1V8#0 -> output:SIM_CARD0
- U$411: device output:#_3V3#0 -> output:VOLTAGE_LEVEL0
- U$412: device output:#_VIN#0 -> output:TEST_POINTS0
- U$413: device output:#_CTS#0 -> output:PTH_PADS0
- U$414: device output:#_RTS#0 -> output:1#8V0
- U$415: device output:#_CLK#0 -> output:3#3V0
- U$416: device output:#_WA#0 -> output:UART20
- U$417: device output:LTE_STICK0 -> output:GPIO0
- U$418: device output:#SHLD#0 -> output:I2C0
- U$419: device output:#DTR#0 -> output:#_#ON##0
- U$420: device output:PWR0 -> output:ON0
- U$421: device output:#_#RST##0 -> output:ON0
- U$422: device SparkFun-Aesthetics:SFE_LOGO_FLAME_.2 -> output:#ON_LED#0
- U$423: device output:LARA#R60 -> output:#PWR_LED#0
- U$424: device output:LARA#R60 -> output:ANT10
- U$425: device output:#RTS_#0 -> output:ANT10
- U$426: device output:#CTS_#0 -> output:ANT20
- U$427: device output:##RESET#_#0 -> output:ANT20
- U$428: device output:##PWR_ON#_#0 -> output:LTE_STICK0
- U$429: device output:#_RXA#0 -> output:#_3V3#0
- U$430: device output:#_TXA#0 -> output:#_GND#0
- U$431: device output:#_TXD#0 -> output:#_GND#0
- U$432: device output:#_RXD#0 -> output:#GND_#0
- U$433: device output:#RXD_#0 -> output:#GND_#0
- U$434: device output:#TXD_#0 -> output:#3V3_#0
- U$435: device output:#RXA_#0 -> output:#VIN_#0
- U$436: device output:#TXA_#0 -> output:#3V3_#0
- U$437: device output:#CLK_#0 -> output:#1V8_#0
- U$438: device output:#WA_#0 -> output:#_1V8#0
- U$439: device output:UART0 -> output:#_3V3#0
- U$440: device output:I2S0 -> output:#_VIN#0
- U$441: device output:ORIENTATION0 -> output:#_CTS#0
- U$442: device output:RST0 -> output:#_RTS#0
- U$443: device output:SIM_CARD0 -> output:#_CLK#0
- U$444: device output:VOLTAGE_LEVEL0 -> output:#_WA#0
- U$445: device output:TEST_POINTS0 -> output:LTE_STICK0
- U$446: device output:PTH_PADS0 -> output:#SHLD#0
- U$447: device output:1#8V0 -> output:#DTR#0
- U$448: device output:3#3V0 -> output:PWR0
- U$449: device output:UART20 -> output:#_#RST##0
- U$450: device output:GPIO0 -> SparkFun-Aesthetics:SFE_LOGO_FLAME_.2
- U$451: device output:I2C0 -> output:LARA#R60
- U$452: device output:#_#ON##0 -> output:LARA#R60
- U$453: device output:ON0 -> output:#RTS_#0
- U$454: device output:ON0 -> output:#CTS_#0
- U$455: device output:#ON_LED#0 -> output:##RESET#_#0
- U$456: device output:#PWR_LED#0 -> output:##PWR_ON#_#0
- U$55: device output:#_GND#0 -> output:LTE_STICK0
- U$61: device output:#_GND#0 -> output:ANT20
- U$62: device output:#GND_#0 -> output:ANT20
- U$63: device output:#GND_#0 -> output:#_3V3#0
- U$64: device output:#3V3_#0 -> output:#_GND#0
- U$65: device output:#VIN_#0 -> output:#_GND#0
- U$66: device output:#3V3_#0 -> output:#GND_#0
- U$67: device output:#1V8_#0 -> output:#GND_#0
- U$68: device output:#_1V8#0 -> output:#3V3_#0
- U$69: device output:#_3V3#0 -> output:#VIN_#0
- U$70: device output:#_VIN#0 -> output:#3V3_#0
- U$71: device output:#_CTS#0 -> output:#1V8_#0
- U$72: device output:#_RTS#0 -> output:#_1V8#0
- U$73: device output:#_CLK#0 -> output:#_3V3#0
- U$74: device output:#_WA#0 -> output:#_VIN#0
- U$75: device output:LTE_STICK0 -> output:#_CTS#0
- U$76: device output:#SHLD#0 -> output:#_RTS#0
- U$77: device output:#DTR#0 -> output:#_CLK#0
- U$78: device output:PWR0 -> output:#_WA#0
- U$79: device output:#_#RST##0 -> output:LTE_STICK0
- U$80: device SparkFun-Aesthetics:SFE_LOGO_FLAME_.2 -> output:#SHLD#0
- U$81: device output:LARA#R60 -> output:#DTR#0
- U$82: device output:LARA#R60 -> output:PWR0
- U$83: device output:#RTS_#0 -> output:#_#RST##0
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Other:
- board text added: "v11"
- board text removed: "v10"
